File: hardware/keyboard_r0/key_switches.kicad_sch (KiCad schematic)
At the start: 126 parts

Commit message: Use custom copy of SW_Push_Dual symbol.
Parts:
- SW_0:0, SW_0:1, SW_0:2, SW_0:3, SW_0:4, SW_0:5, SW_0:6, SW_1:0, SW_1:1, SW_1:2, SW_1:3, SW_1:4, SW_1:5, SW_1:6, SW_2:0, SW_2:1, SW_2:2, SW_2:3, SW_2:4, SW_2:5, SW_3:0, SW_3:1, SW_3:2, SW_3:3, SW_3:4, SW_3:5, SW_3:6, SW_4:0, SW_4:1, SW_4:2, SW_4:3, SW_4:4, SW_T0:2, SW_T0:3, SW_T1:1, SW_T1:2, SW_T1:3, SW_T2:3, SW_T3:0, SW_T3:1, SW_T3:2, SW_T3:3: symbol Switch:SW_Push_Dual -> mass:SW_Push_Dual
Changed lines of the file:
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@@
 	)
 	(symbol
-		(lib_id "Switch:SW_Push_Dual")
+		(lib_id "mass:SW_Push_Dual")
 		(at 101.6 83.82 0)
 		(unit 1)
@@
 	)
 	(symbol
-		(lib_id "Switch:SW_Push_Dual")
+		(lib_id "mass:SW_Push_Dual")
 		(at 101.6 160.02 0)
 		(unit 1)
@@
 	)
 	(symbol
-		(lib_id "Switch:SW_Push_Dual")
+		(lib_id "mass:SW_Push_Dual")
 		(at 203.2 109.22 0)
 		(unit 1)
@@
 	)
 	(symbol
-		(lib_id "Switch:SW_Push_Dual")
+		(lib_id "mass:SW_Push_Dual")
 		(at 76.2 58.42 0)
 		(unit 1)
@@
 	)
 	(symbol
-		(lib_id "Switch:SW_Push_Dual")
+		(lib_id "mass:SW_Push_Dual")
 		(at 101.6 33.02 0)
 		(unit 1)
@@
 	)
 	(symbol
-		(lib_id "Switch:SW_Push_Dual")
+		(lib_id "mass:SW_Push_Dual")
 		(at 152.4 109.22 0)
 		(unit 1)
@@
 	)
 	(symbol
-		(lib_id "Switch:SW_Push_Dual")
+		(lib_id "mass:SW_Push_Dual")
 		(at 127 33.02 0)
 		(unit 1)
@@
 	)
 	(symbol
-		(lib_id "Switch:SW_Push_Dual")
+		(lib_id "mass:SW_Push_Dual")
 		(at 127 58.42 0)
 		(unit 1)
@@
 	)
 	(symbol
-		(lib_id "Switch:SW_Push_Dual")
+		(lib_id "mass:SW_Push_Dual")
 		(at 203.2 160.02 0)
 		(unit 1)
@@
 	)
 	(symbol
-		(lib_id "Switch:SW_Push_Dual")
+		(lib_id "mass:SW_Push_Dual")
 		(at 152.4 58.42 0)
 		(unit 1)
@@
 	)
 	(symbol
-		(lib_id "Switch:SW_Push_Dual")
+		(lib_id "mass:SW_Push_Dual")
 		(at 152.4 33.02 0)
 		(unit 1)
@@
 	)
 	(symbol
-		(lib_id "Switch:SW_Push_Dual")
+		(lib_id "mass:SW_Push_Dual")
 		(at 127 109.22 0)
 		(unit 1)
@@
 	)
 	(symbol
-		(lib_id "Switch:SW_Push_Dual")
+		(lib_id "mass:SW_Push_Dual")
 		(at 177.8 33.02 0)
 		(unit 1)
@@
 	)
 	(symbol
-		(lib_id "Switch:SW_Push_Dual")
+		(lib_id "mass:SW_Push_Dual")
 		(at 101.6 58.42 0)
 		(unit 1)
@@
 	)
 	(symbol
-		(lib_id "Switch:SW_Push_Dual")
+		(lib_id "mass:SW_Push_Dual")
 		(at 177.8 134.62 0)
 		(unit 1)
@@
 	)
 	(symbol
-		(lib_id "Switch:SW_Push_Dual")
+		(lib_id "mass:SW_Push_Dual")
 		(at 177.8 83.82 0)
 		(unit 1)
@@
 	)
 	(symbol
-		(lib_id "Switch:SW_Push_Dual")
+		(lib_id "mass:SW_Push_Dual")
 		(at 203.2 134.62 0)
 		(unit 1)
@@
 	)
 	(symbol
-		(lib_id "Switch:SW_Push_Dual")
+		(lib_id "mass:SW_Push_Dual")
 		(at 152.4 134.62 0)
 		(unit 1)
@@
 	)
 	(symbol
-		(lib_id "Switch:SW_Push_Dual")
+		(lib_id "mass:SW_Push_Dual")
 		(at 152.4 83.82 0)
 		(unit 1)
@@
 	)
 	(symbol
-		(lib_id "Switch:SW_Push_Dual")
+		(lib_id "mass:SW_Push_Dual")
 		(at 101.6 134.62 0)
 		(unit 1)
@@
 	)
 	(symbol
-		(lib_id "Switch:SW_Push_Dual")
+		(lib_id "mass:SW_Push_Dual")
 		(at 50.8 134.62 0)
 		(unit 1)
@@
 	)
 	(symbol
-		(lib_id "Switch:SW_Push_Dual")
+		(lib_id "mass:SW_Push_Dual")
 		(at 203.2 58.42 0)
 		(unit 1)
@@
 	)
 	(symbol
-		(lib_id "Switch:SW_Push_Dual")
+		(lib_id "mass:SW_Push_Dual")
 		(at 101.6 109.22 0)
 		(unit 1)
@@
 	)
 	(symbol
-		(lib_id "Switch:SW_Push_Dual")
+		(lib_id "mass:SW_Push_Dual")
 		(at 50.8 109.22 0)
 		(unit 1)
@@
 	)
 	(symbol
-		(lib_id "Switch:SW_Push_Dual")
+		(lib_id "mass:SW_Push_Dual")
 		(at 50.8 83.82 0)
 		(unit 1)
@@
 	)
 	(symbol
-		(lib_id "Switch:SW_Push_Dual")
+		(lib_id "mass:SW_Push_Dual")
 		(at 76.2 83.82 0)
 		(unit 1)
@@
 	)
 	(symbol
-		(lib_id "Switch:SW_Push_Dual")
+		(lib_id "mass:SW_Push_Dual")
 		(at 76.2 160.02 0)
 		(unit 1)
@@
 	)
 	(symbol
-		(lib_id "Switch:SW_Push_Dual")
+		(lib_id "mass:SW_Push_Dual")
 		(at 177.8 160.02 0)
 		(unit 1)
@@
 	)
 	(symbol
-		(lib_id "Switch:SW_Push_Dual")
+		(lib_id "mass:SW_Push_Dual")
 		(at 177.8 109.22 0)
 		(unit 1)
@@
 	)
 	(symbol
-		(lib_id "Switch:SW_Push_Dual")
+		(lib_id "mass:SW_Push_Dual")
 		(at 127 83.82 0)
 		(unit 1)
@@
 	)
 	(symbol
-		(lib_id "Switch:SW_Push_Dual")
+		(lib_id "mass:SW_Push_Dual")
 		(at 152.4 160.02 0)
 		(unit 1)
@@
 	)
 	(symbol
-		(lib_id "Switch:SW_Push_Dual")
+		(lib_id "mass:SW_Push_Dual")
 		(at 50.8 33.02 0)
 		(unit 1)
@@
 	)
 	(symbol
-		(lib_id "Switch:SW_Push_Dual")
+		(lib_id "mass:SW_Push_Dual")
 		(at 203.2 83.82 0)
 		(unit 1)
@@
 	)
 	(symbol
-		(lib_id "Switch:SW_Push_Dual")
+		(lib_id "mass:SW_Push_Dual")
 		(at 50.8 58.42 0)
 		(unit 1)
@@
 	)
 	(symbol
-		(lib_id "Switch:SW_Push_Dual")
+		(lib_id "mass:SW_Push_Dual")
 		(at 50.8 160.02 0)
 		(unit 1)
@@
 	)
 	(symbol
-		(lib_id "Switch:SW_Push_Dual")
+		(lib_id "mass:SW_Push_Dual")
 		(at 76.2 134.62 0)
 		(unit 1)
@@
 	)
 	(symbol
-		(lib_id "Switch:SW_Push_Dual")
+		(lib_id "mass:SW_Push_Dual")
 		(at 127 134.62 0)
 		(unit 1)
@@
 	)
 	(symbol
-		(lib_id "Switch:SW_Push_Dual")
+		(lib_id "mass:SW_Push_Dual")
 		(at 76.2 33.02 0)
 		(unit 1)
@@
 	)
 	(symbol
-		(lib_id "Switch:SW_Push_Dual")
+		(lib_id "mass:SW_Push_Dual")
 		(at 203.2 33.02 0)
 		(unit 1)
@@
 	)
 	(symbol
-		(lib_id "Switch:SW_Push_Dual")
+		(lib_id "mass:SW_Push_Dual")
 		(at 177.8 58.42 0)
 		(unit 1)
@@
 	)
 	(symbol
-		(lib_id "Switch:SW_Push_Dual")
+		(lib_id "mass:SW_Push_Dual")
 		(at 127 160.02 0)
 		(unit 1)
@@
 	)
 	(symbol
-		(lib_id "Switch:SW_Push_Dual")
+		(lib_id "mass:SW_Push_Dual")
 		(at 76.2 109.22 0)
 		(unit 1)
